File: PCB/pressure_pad.kicad_sch (KiCad schematic)
At the start: 52 parts, among them J1 MULTIPLEXER INPUTS, J2 DEMULTIPLEXER OUTPUTS

Commit message: docs
Other:
- title: Presure Pad Data Collection Circuit Schematic -> Pressure Pad Data Collection Circuit Schematic
Changed lines of the file:
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@@
 	(paper "A4")
 	(title_block
-		(title "Presure Pad Data Collection Circuit Schematic")
+		(title "Pressure Pad Data Collection Circuit Schematic")
 		(date "2025-07-07")
 		(rev "7")
