File: OLD/PCB/pressure_pad.kicad_sch (KiCad schematic)
At the start: 52 parts, among them J1 MULTIPLEXER INPUTS, J2 DEMULTIPLEXER OUTPUTS

Commit message: next
Connections:
- net SDA: no longer A1.D20 (D20/SDA), DEMUX1.3 (SDA), DEMUX2.3 (SDA), DEMUX3.3 (SDA), DEMUX4.3 (SDA), MUX1.3 (SDA), MUX3.3 (SDA), R8.1
- net SCL renamed SCL1
- new net SDA1: A1.D20 (D20/SDA), DEMUX1.3 (SDA), DEMUX2.3 (SDA), DEMUX3.3 (SDA), DEMUX4.3 (SDA), MUX1.3 (SDA), MUX3.3 (SDA), R8.1
Other:
- title: Pressure Pad Data Collection Circuit Schematic -> Pressure Pad Data Collection Circuit Schematic (v2)
